Commit message: complete urdf model(without lidars)

File: dev_ws/src/schaeffler_robot_urdf/urdf/corrected_robot_core.xacro (robot description, xacro)
@@ -16,4 +16,5 @@
     <!-- BASE LINK -->
     <link name="base_link">
+	<origin xyz="0 0 0" />
     </link>
     <!-- CHASSIS LINK -->
@@ -21,22 +22,22 @@
         <parent link="base_link" />
         <child link="chassis" />
-        <origin xyz="-0.5 0 0" />
+        <origin xyz="-0.5 0 -0.025" />
     </joint>
     <link name="chassis">
         <visual>
-            <origin xyz="0.5 0 0.05" />
+            <origin xyz="0.5 0 0.1" />
             <geometry>
-                <box size="1 0.7 0.1" />
+                <box size="1 0.7 0.2" />
             </geometry>
             <material name="white" />
         </visual>
         <collision>
-            <origin xyz="0.5 0 0.05" />
+            <origin xyz="0.5 0 0" />
             <geometry>
-                <box size="1 0.7 0.1" />
+                <box size="1 0.7 0.2" />
             </geometry>
         </collision>
-        <xacro:inertial_box mass="50" x="1" y="0.7" z="0.1">
-            <origin xyz="0.5 0 0.05" rpy="0 0 0" />
+        <xacro:inertial_box mass="50" x="1" y="0.7" z="0.2">
+            <origin xyz="0 0 0" rpy="0 0 0" />
         </xacro:inertial_box>
     </link>
@@ -87,3 +88,92 @@
         </xacro:inertial_cylinder>
     </link>
+    <!-- CASTER WHEEL LINKS -->
+    <!-- caster_wheel_joint_fl LINK -->
+    <joint name="caster_wheel_joint_fl" type="fixed">
+        <parent link="chassis" />
+        <child link="caster_wheel_fl" />
+        <origin xyz="0.9 0.3 -0.025" />
+    </joint>
+    <link name="caster_wheel_fl">
+        <visual>
+            <geometry>
+                <sphere radius="0.04"/>
+            </geometry>
+            <material name="black" />
+        </visual>
+	<collision>
+            <geometry>
+                <sphere radius="0.04"/>
+            </geometry>
+        </collision>
+	 <xacro:inertial_sphere mass="1" radius="0.04">
+            <origin xyz="0 0 0" rpy="0 0 0" />
+        </xacro:inertial_sphere>
+    </link>
+ <!-- caster_wheel_joint_fr LINK -->
+    <joint name="caster_wheel_joint_fr" type="fixed">
+        <parent link="chassis" />
+        <child link="caster_wheel_fr" />
+        <origin xyz="0.9 -0.3 -0.025" />
+    </joint>
+    <link name="caster_wheel_fr">
+        <visual>
+            <geometry>
+                <sphere radius="0.04"/>
+            </geometry>
+            <material name="black" />
+        </visual>
+	<collision>
+            <geometry>
+                <sphere radius="0.04"/>
+            </geometry>
+        </collision>
+	<xacro:inertial_sphere mass="1" radius="0.04">
+            <origin xyz="0 0 0" rpy="0 0 0" />
+        </xacro:inertial_sphere>
+    </link>
+ <!-- caster_wheel_joint_bl LINK -->
+    <joint name="caster_wheel_joint_bl" type="fixed">
+        <parent link="chassis" />
+        <child link="caster_wheel_bl" />
+        <origin xyz="0.1 0.3 -0.025" />
+    </joint>
+    <link name="caster_wheel_bl">
+        <visual>
+            <geometry>
+                <sphere radius="0.04"/>
+            </geometry>
+            <material name="black" />
+        </visual>
+	<collision>
+            <geometry>
+                <sphere radius="0.04"/>
+            </geometry>
+        </collision>
+`	<xacro:inertial_sphere mass="1" radius="0.04">
+            <origin xyz="0 0 0" rpy="0 0 0" />
+        </xacro:inertial_sphere>
+    </link>
+ <!-- caster_wheel_joint_br LINK -->
+    <joint name="caster_wheel_joint_br" type="fixed">
+        <parent link="chassis" />
+        <child link="caster_wheel_br" />
+        <origin xyz="0.1 -0.3 -0.025" />
+    </joint>
+    <link name="caster_wheel_br">
+        <visual>
+            <geometry>
+                <sphere radius="0.04"/>
+            </geometry>
+            <material name="black" />
+        </visual>
+	<collision>
+            <geometry>
+                <sphere radius="0.04"/>
+            </geometry>
+        </collision>
+	<xacro:inertial_sphere mass="1" radius="0.04">
+            <origin xyz="0 0 0" rpy="0 0 0" />
+        </xacro:inertial_sphere>
+    </link>
 </robot>

File: dev_ws/src/schaeffler_robot_urdf/urdf/robot_core.xacro (robot description, xacro)
@@ -28,12 +28,12 @@
             <origin xyz="0.5 0 0.05">
             <geometry>
-                <box size="1 0.7 0.1" />
+                <box size="0.7 1 0.1" />
             </geometry>
             <material name="white"/>
         </visual>
         <collision>
-            <origin xyz="0.5 0 0.05">
+            <origin xyz="0 0 0">
             <geometry>
-                <box size="1 0.7 0.1" />
+                <box size="0.7 1 0.1" />
             </geometry>
         </collision>
@@ -62,5 +62,5 @@
         </collision>
         <xacro:inertial_cylinder mass="5" length="0.04" radius="0.08">
-          <!--  </origin xyz="0 0 0" rpy="0 0 0" /> -->
+         </origin xyz="0 0 0" rpy="0 0 0" />
         </xacro:inertial_cylinder>
     </link>
@@ -85,5 +85,5 @@
         </collision>
         <xacro:inertial_cylinder mass="5" length="0.04" radius="0.08">
-          <!--  </origin xyz="0 0 0" rpy="0 0 0" /> -->
+          </origin xyz="0 0 0" rpy="0 0 0" />
         </xacro:inertial_cylinder>
     </link>

Commit message: start of gazebo/lidar

File: dev_ws/src/schaeffler_robot_urdf/urdf/corrected_robot_core.xacro (robot description, xacro)
@@ -14,4 +14,7 @@
         <color rgba="0 0 0 1" />
     </material>
+    <material name="red">
+        <color rgba="1 0 0 1" />
+    </material>
     <!-- BASE LINK -->
     <link name="base_link">
@@ -33,5 +36,5 @@
         </visual>
         <collision>
-            <origin xyz="0.5 0 0" />
+            <origin xyz="0.5 0 0.1" />
             <geometry>
                 <box size="1 0.7 0.2" />
@@ -42,4 +45,7 @@
         </xacro:inertial_box>
     </link>
+    <gazebo reference="chassis">
+	<material>Gazebo/white</material>
+    </gazebo>
     <!-- LEFT WHEEL LINK -->
     <joint name="left_wheel_joint" type="continuous">
@@ -65,4 +71,7 @@
         </xacro:inertial_cylinder>
     </link>
+    <gazebo reference="left_wheel">
+	<material>Gazebo/blue</material>
+    </gazebo>
     <!-- RIGHT WHEEL LINK -->
     <joint name="right_wheel_joint" type="continuous">
@@ -88,4 +97,7 @@
         </xacro:inertial_cylinder>
     </link>
+    <gazebo reference="right_wheel">
+	<material>Gazebo/blue</material>
+    </gazebo>
     <!-- CASTER WHEEL LINKS -->
     <!-- caster_wheel_joint_fl LINK -->
@@ -111,4 +123,7 @@
         </xacro:inertial_sphere>
     </link>
+    <gazebo reference="caster_wheel_fl">
+	<material>Gazebo/black</material>
+    </gazebo>
  <!-- caster_wheel_joint_fr LINK -->
     <joint name="caster_wheel_joint_fr" type="fixed">
@@ -133,4 +148,7 @@
         </xacro:inertial_sphere>
     </link>
+    <gazebo reference="caster_wheel_fr">
+	<material>Gazebo/black</material>
+    </gazebo>
  <!-- caster_wheel_joint_bl LINK -->
     <joint name="caster_wheel_joint_bl" type="fixed">
@@ -155,4 +173,7 @@
         </xacro:inertial_sphere>
     </link>
+    <gazebo reference="caster_wheel_bl">
+	<material>Gazebo/black</material>
+    </gazebo>
  <!-- caster_wheel_joint_br LINK -->
     <joint name="caster_wheel_joint_br" type="fixed">
@@ -177,3 +198,6 @@
         </xacro:inertial_sphere>
     </link>
+    <gazebo reference="caster_wheel_br">
+	<material>Gazebo/black</material>
+    </gazebo>
 </robot>

File: dev_ws/src/schaeffler_robot_urdf/urdf/robot.urdf.xacro (robot description, xacro)
@@ -2,3 +2,5 @@
 <robot xmlns:xacro="http://www.ros.org/wiki/xacro" name="robot">
     <xacro:include filename="corrected_robot_core.xacro"/>
+    <xacro:include filename="lidar.xacro"/>
+    <xacro:include filename="gazebo_control.xarco"/>
 </robot>

File: dev_ws/src/sick_tim/urdf/sick_tim.urdf.xacro (robot description, xacro)
@@ -1,5 +1,5 @@
 <?xml version="1.0"?>
 <robot xmlns:xacro="http://ros.org/wiki/xacro">
-  <xacro:macro name="sick_tim310" params="name ros_topic min_angle:=-2.357 max_angle:=2.357 min_range:=0.05 max_range:=4.0">
+  <xacro:macro name="sick_tim310" params="name ros_topic min_angle:=-2.357 max_angle:=2.357 min_range:=0.05 max_range:=10.0">
     <xacro:sick_tim name="${name}" ros_topic="${ros_topic}"
       length="0.06" width="0.06" height="0.079" mass="0.150" z_offset="0.05595"
